Commit message: upd: create bringup pkg for launch stack on real robot

File: src/asump_description/urdf/lidar.xacro (robot description, xacro)
@@ -2,5 +2,5 @@
 <robot xmlns:xacro="http://www.ros.org/wiki/xacro">
   <xacro:macro name="lidar" params="parent_link x y z roll pitch yaw">
-    <link name="lidar_link">
+    <link name="laser">
       <inertial>
         <origin xyz="-0.391109515510156 1.97239805683526E-07 -0.302515275293891" rpy="0 0 0"/>
@@ -26,5 +26,5 @@
       <origin xyz="${x} ${y} ${z}" rpy="${roll} ${pitch} ${yaw}"/>
       <parent link="${parent_link}"/>
-      <child link="lidar_link"/>
+      <child link="laser"/>
       <axis xyz="0 0 0"/>
     </joint>
@@ -32,5 +32,5 @@
     <joint name="lidar_ray_joint" type="fixed">
       <origin xyz="0 0 0.02" rpy="0 0 0"/>
-      <parent link="lidar_link"/>
+      <parent link="laser"/>
       <child link="lidar_ray_link"/>
       <axis xyz="0 0 0"/>

File: src/asump_description/urdf/robot.xacro (robot description, xacro)
@@ -14,5 +14,5 @@
     parent_link="base_link"
     x="0.496510223719" y="0" z="0.596484004557"
-    roll="0" pitch="0" yaw="0"
+    roll="0" pitch="0" yaw="-3.14"
   />
   <xacro:rlai_depth_camera
