Commit message: upd: remake sim wirld and fix rollers of robot

File: src/asump_description/urdf/base_link.xacro (robot description, xacro)
@@ -40,5 +40,5 @@
                iyy="31.0730345912135" iyz="0.00228580331928839" izz="29.139821759891"/>
     </inertial>
-    <visual>
+    <!--visual>
       <origin xyz="0 0 0" rpy="0 0 0"/>
       <geometry>
@@ -46,5 +46,5 @@
       </geometry>
       <material name=""><color rgba="0 0 0 1"/></material>
-    </visual>
+    </visual-->
   </link>
   <joint name="tracks_joint" type="fixed">

File: src/asump_description/urdf/roller_params.xacro (robot description, xacro)
@@ -10,15 +10,15 @@
                  iyy="0.00353589020904659" iyz="-3.27203986802643E-19" izz="0.00179016454216458"/>
       </inertial>
-      <!--visual>
+      <visual>
         <origin xyz="0 0 0" rpy="0 0 0"/>
         <geometry>
-          <mesh filename="file://$(find asump_description)/meshes/${name}_roller.STL"/>
+          <mesh filename="file://$(find asump_description)/meshes/${name}_roller.STL" scale="1 0.5 1"/>
         </geometry>
-        <material name=""><color rgba="0.564705882352941 0.564705882352941 0.564705882352941 0"/></material>
-      </visual-->
+        <material name=""><color rgba="0.564705882352941 0.564705882352941 0.564705882352941 1"/></material>
+      </visual>
       <collision>
         <origin xyz="0 0 0" rpy="0 0 0"/>
         <geometry>
-          <mesh filename="file://$(find asump_description)/meshes/${name}_roller.STL"/>
+          <mesh filename="file://$(find asump_description)/meshes/${name}_roller.STL" scale="1 0.5 1"/>
         </geometry>
       </collision>
@@ -29,21 +29,13 @@
       <child link="${name}_roller"/>
       <axis xyz="${axis_x} ${axis_y} ${axis_z}"/>
-      <limit effort="1000" velocity="10"/>
-      <dynamics friction="0.5"/>
+      <limit effort="500" velocity="10"/>
+      <dynamics friction="0.2"/>
     </joint>
     <gazebo reference="${name}_roller">
-      <visual>
-        <cast_shadows>false</cast_shadows>
-        <transparency>1.0</transparency>
-      </visual>
       <!-- Настройки трения с поверхностью -->
-      <mu1>0.1</mu1>        <!-- Коэффициент трения в продольном направлении -->
-      <mu2>0.2</mu2>        <!-- Коэффициент трения в поперечном направлении -->
+      <mu1>0.4</mu1>        <!-- Коэффициент трения в продольном направлении -->
+      <mu2>0.1</mu2>        <!-- Коэффициент трения в поперечном направлении -->
       <kp>1e5</kp>          <!-- Коэффициент жесткости контакта -->
       <kd>1e3</kd>          <!-- Коэффициент демпфирования контакта -->
-      <collision>
-        <laser_retro>0</laser_retro>
-        <max_contacts>10</max_contacts>
-      </collision>
     </gazebo>
   </xacro:macro>

Commit message: upd: add depth_camera for publish pontcloud to sim and balance weidth block

File: src/asump_description/urdf/base_link.xacro (robot description, xacro)
@@ -8,5 +8,5 @@
     <inertial>
       <origin xyz="0.109332549621884 -3.99444698804471E-06 0.303288060337734" rpy="0 0 0"/>
-      <mass value="2.5"/>
+      <mass value="7.5"/>
       <inertia ixx="13.4992891087176" ixy="0.000473313057343369" ixz="-1.40847406797442"
                iyy="29.2623362046841" iyz="0.00234656617180413" izz="27.4848319406113"/>
@@ -30,4 +30,18 @@
     <parent link="base_footprint"/>
     <child link="base_link"/>
+    <axis xyz="0 0 0"/>
+  </joint>
+  <link name="balance_link">
+    <inertial>
+      <origin xyz="0 0 0" rpy="0 0 0"/>
+      <mass value="3.2"/>
+      <inertia ixx="13.4992891087176" ixy="0.000473313057343369" ixz="-1.40847406797442"
+               iyy="29.2623362046841" iyz="0.00234656617180413" izz="27.4848319406113"/>
+    </inertial>
+  </link>
+  <joint name="balance_joint" type="fixed">
+    <origin xyz="0 0 0.25" rpy="0 0 0"/>
+    <parent link="base_link"/>
+    <child link="balance_link"/>
     <axis xyz="0 0 0"/>
   </joint>

File: src/asump_description/urdf/depth_camera.xacro (robot description, xacro)
@@ -12,7 +12,7 @@
     <link name="depth_camera_link">
       <visual>
-        <origin xyz="0 0 0" rpy="0 0 0"/>
+        <origin xyz="0 0 0" rpy="${-pi/2} 0 0"/>
         <geometry>
-          <mesh filename="file://$(find asump_description)/meshes/depth_camera_housing.stl" scale="0.001 0.001 0.001"/>
+          <mesh filename="package://realsense2_description/meshes/d415.stl"/>
         </geometry>
         <material name="camera_dark_gray">
@@ -26,9 +26,8 @@
         </geometry>
       </collision>
-      <inertial>
+      <!--inertial>
         <mass value="0.072"/>
-        <!-- Thin bar — treat as box: m(b²+c²)/12 etc. -->
         <inertia ixx="0.000010" ixy="0" ixz="0" iyy="0.000010" iyz="0" izz="0.000010"/>
-      </inertial>
+      </inertial-->
     </link>
     <joint name="depth_camera_joint" type="fixed">
@@ -62,9 +61,9 @@
         </material>
       </visual>
-      <sensor name="depth_camera" type="depth_camera">
+      <sensor name="depth_camera" type="rgbd_camera">
         <always_on>true</always_on>
         <update_rate>30</update_rate>
         <topic>/depth_camera/depth</topic>
-        <gz_frame_id>depth_camera_depth_optical_frame</gz_frame_id>
+        <gz_frame_id>depth_camera_link</gz_frame_id>
         <camera name="depth_camera">
           <horizontal_fov>1.5184</horizontal_fov>
@@ -85,5 +84,5 @@
         </camera>
       </sensor>
-      <sensor name="rgb_camera" type="camera">
+      <!--sensor name="rgb_camera" type="camera">
         <always_on>true</always_on>
         <update_rate>30</update_rate>
@@ -107,5 +106,5 @@
           </noise>
         </camera>
-      </sensor>
+      </sensor-->
     </gazebo>
   </xacro:macro>

File: src/asump_description/urdf/robot.xacro (robot description, xacro)
@@ -9,4 +9,5 @@
   <xacro:include filename="gazebo_control.xacro"/>
   <xacro:include filename="depth_camera.xacro"/>
+  <!--xacro:include filename="d415.xacro"/-->
   <xacro:property name="robot_name" value="asump0"/>
   <xacro:lidar
@@ -17,8 +18,13 @@
   <xacro:rlai_depth_camera
     parent="base_link"
-    xyz="0.648 0 0.253"
+    xyz="0.648 0 0.24"
     rpy="0 0 0"
     model="$(arg camera_model)"
   />
+  <!--xacro:simple_d415_camera
+    parent="base_link"
+    xyz="0.648 0.0 0.24"
+    rpy="0 0 0"
+    name="depth_camera"/-->
   <!-- Установка камер
   <xacro:left_parking_sensor parent_link="base_link" x="-0.25577" y="0.26863" z="0.46916" roll="0" pitch="-0.087266" yaw="1.5708"/>

File: src/asump_description/urdf/roller_params.xacro (robot description, xacro)
@@ -6,5 +6,5 @@
       <inertial>
         <origin xyz="0 -0.01 0" rpy="0 0 0"/>
-        <mass value="0.65"/>
+        <mass value="1.2"/>
         <inertia ixx="0.00179016454216459" ixy="1.32679515530007E-36" ixz="1.04242882131926E-50"
                  iyy="0.00353589020904659" iyz="-3.27203986802643E-19" izz="0.00179016454216458"/>
@@ -29,5 +29,5 @@
       <child link="${name}_roller"/>
       <axis xyz="${axis_x} ${axis_y} ${axis_z}"/>
-      <limit effort="500" velocity="10"/>
+      <limit effort="25000" velocity="100"/>
       <dynamics friction="0.2"/>
     </joint>

Commit message: upd: try to use amcl instead of slam_toolbox

File: src/asump_description/urdf/base_link.xacro (robot description, xacro)
@@ -47,5 +47,5 @@
   </joint>
   <!-- Траки -->
-  <link name="tracks_link">
+  <!--link name="tracks_link">
     <inertial>
       <origin xyz="0.105400708208844 1.85139805717996E-07 0.293968729263109" rpy="0 0 0"/>
@@ -54,5 +54,5 @@
                iyy="31.0730345912135" iyz="0.00228580331928839" izz="29.139821759891"/>
     </inertial>
-    <!--visual>
+    <visual>
       <origin xyz="0 0 0" rpy="0 0 0"/>
       <geometry>
@@ -60,5 +60,5 @@
       </geometry>
       <material name=""><color rgba="0 0 0 1"/></material>
-    </visual-->
+    </visual>
   </link>
   <joint name="tracks_joint" type="fixed">
@@ -70,5 +70,5 @@
   <gazebo reference="tracks_link">
     <material>Gazebo/Black</material>
-  </gazebo>
+  </gazebo-->
   <!-- Ролики -->
   <xacro:roller name="fl" x="0.30749" y="0.25132" z="0.079492" axis_x="0" axis_y="1" axis_z="0"/>
