Commit message: upd: preready state for mapping test

File: src/asump_description/urdf/robot1.xacro (robot description, xacro)
@@ -2,4 +2,5 @@
 <robot name="surfex_robot" xmlns:xacro="http://www.ros.org/wiki/xacro">
   <xacro:include filename="$(find realsense2_description)/urdf/_d435.urdf.xacro" />
+  <link name="base_footprint"/>
   <link name="base_link">
     <inertial>
@@ -11,5 +12,5 @@
       <origin xyz="0 0 0" rpy="1.5708 0 -1.5708"/>
       <geometry>
-        <mesh filename="file://$(find asump_description)/meshes/base_link1.stl" scale="0.001 0.001 0.001"/>
+        <mesh filename="file://$(find asump_description)/meshes/base_link.stl" scale="0.001 0.001 0.001"/>
       </geometry>
       <material name=""><color rgba="0.1 0.1 0.1 1"/></material>
@@ -18,8 +19,13 @@
       <origin xyz="0 0 0" rpy="1.5708 0 -1.5708"/>
       <geometry>
-        <mesh filename="file://$(find asump_description)/meshes/base_link1.stl" scale="0.001 0.001 0.001"/>
-      </geometry>
-    </collision>
-  </link>
+        <mesh filename="file://$(find asump_description)/meshes/base_link.stl" scale="0.001 0.001 0.001"/>
+      </geometry>
+    </collision>
+  </link>
+  <joint name="base_footprint_joint" type="fixed">
+    <parent link="base_footprint"/>
+    <child link="base_link"/>
+    <origin xyz="0.0 0.0 0.0" rpy="0 0 0"/>
+  </joint>
   <link name="body_link">
     <inertial>
@@ -68,4 +74,58 @@
     <origin xyz="0.4625 0.0 0.0" rpy="0 0 0"/>
   </joint>
+  <link name="face_left_us_sensor_link">
+    <inertial>
+      <origin xyz="0 0 0" rpy="0 0 0"/>
+      <mass value="0.0437"/>
+      <inertia ixx="1.591e-5" ixy="0.0" ixz="-1.311e-6"
+               iyy="1.267e-5" iyz="0.0"
+               izz="1.167e-5"/>
+    </inertial>
+    <visual>
+      <origin xyz="0 0 0" rpy="0 0 0"/>
+      <geometry>
+        <mesh filename="file://$(find asump_description)/meshes/ultrasonic_sensor.stl" scale="0.001 0.001 0.001"/>
+      </geometry>
+      <material name=""><color rgba="0.2 0.2 0.2 1.0"/></material>
+    </visual>
+    <collision>
+      <origin xyz="0 0 0" rpy="0 0 0"/>
+      <geometry>
+        <mesh filename="file://$(find asump_description)/meshes/ultrasonic_sensor.stl" scale="0.001 0.001 0.001"/>
+      </geometry>
+    </collision>
+  </link>
+  <joint name="face_left_us_sensor_joint" type="fixed">
+    <parent link="face_sensor_panel"/>
+    <child link="face_left_us_sensor_link"/>
+    <origin xyz="0.02845 0.121508 0.018" rpy="0 0.5236 0"/>
+  </joint>
+  <link name="face_right_us_sensor_link">
+    <inertial>
+      <origin xyz="0 0 0" rpy="0 0 0"/>
+      <mass value="0.0437"/>
+      <inertia ixx="1.591e-5" ixy="0.0" ixz="-1.311e-6"
+               iyy="1.267e-5" iyz="0.0"
+               izz="1.167e-5"/>
+    </inertial>
+    <visual>
+      <origin xyz="0 0 0" rpy="0 0 0"/>
+      <geometry>
+        <mesh filename="file://$(find asump_description)/meshes/ultrasonic_sensor.stl" scale="0.001 0.001 0.001"/>
+      </geometry>
+      <material name=""><color rgba="0.2 0.2 0.2 1.0"/></material>
+    </visual>
+    <collision>
+      <origin xyz="0 0 0" rpy="0 0 0"/>
+      <geometry>
+        <mesh filename="file://$(find asump_description)/meshes/ultrasonic_sensor.stl" scale="0.001 0.001 0.001"/>
+      </geometry>
+    </collision>
+  </link>
+  <joint name="face_right_us_sensor_joint" type="fixed">
+    <parent link="face_sensor_panel"/>
+    <child link="face_right_us_sensor_link"/>
+    <origin xyz="0.02845 -0.121508 0.018" rpy="0 0.5236 0"/>
+  </joint>
   <link name="laser">
     <inertial>
@@ -76,10 +136,10 @@
     <visual>
       <origin xyz="0 0 0" rpy="0 0 0"/>
-      <geometry><mesh filename="file://$(find asump_description)/meshes/lidar_link1.stl" scale="0.001 0.001 0.001"/></geometry>
+      <geometry><mesh filename="file://$(find asump_description)/meshes/lidar_link.stl" scale="0.001 0.001 0.001"/></geometry>
       <material name=""><color rgba="0.1 0.1 0.1 1"/></material>
     </visual>
     <collision>
       <origin xyz="0 0 0" rpy="0 0 0"/>
-      <geometry><mesh filename="file://$(find asump_description)/meshes/lidar_link1.stl" scale="0.001 0.001 0.001"/></geometry>
+      <geometry><mesh filename="file://$(find asump_description)/meshes/lidar_link.stl" scale="0.001 0.001 0.001"/></geometry>
     </collision>
   </link>
@@ -89,5 +149,5 @@
     <origin xyz="0.1425 0.0 0.373" rpy="0 0 0"/>
   </joint>
-  <xacro:sensor_d435 parent="face_sensor_panel" name="camera" use_nominal_extrinsics="true">
+  <xacro:sensor_d435 parent="face_sensor_panel" name="face_camera" use_nominal_extrinsics="true">
     <origin xyz="0.02 0.0 0.01" rpy="0 0 0"/>
   </xacro:sensor_d435>
@@ -127,97 +187,203 @@
   <xacro:wheel prefix="rl" xyz="-0.314 0.2519 0" rpy="0 0 0"/>
   <xacro:wheel prefix="rr" xyz="-0.314 -0.2519 0" rpy="0 0 0"/>
-  <!--
-  <link name="lidar_link">
-    <inertial>
-      <origin xyz="-2.94e-07 2.96e-07 0.018590" rpy="0 0 0"/>
-      <mass value="1.274"/>
-      <inertia ixx="0.000577" iyy="0.000577" izz="0.00083" ixy="0.0" iyz="0.0" ixz="0.0"/>
-    </inertial>
-    <visual>
-      <origin xyz="-0.029992 -0.112508 -0.671" rpy="0 0 0"/>
-      <geometry><mesh filename="file://$(find asump_description)/meshes/lidar_link.stl" scale="0.001 0.001 0.001"/></geometry>
-      <material name=""><color rgba="1 1 1 1"/></material>
-    </visual>
-    <collision>
-      <origin xyz="-0.029992 -0.112508 -0.671" rpy="0 0 0"/>
-      <geometry><mesh filename="file://$(find asump_description)/meshes/lidar_link.stl" scale="0.001 0.001 0.001"/></geometry>
-    </collision>
-  </link>
-  <joint name="lidar_joint" type="fixed">
-    <parent link="base_link"/>
-    <child link="lidar_link"/>
-    <origin xyz="0.0 0.0 0.0" rpy="0 0 0"/>
-  </joint>
-  <link name="l1_us_mount">
-    <inertial>
-      <origin xyz="-0.022207 0.474008 -0.301902" rpy="0 0 0"/>
-      <mass value="0.285"/>
-      <inertia ixx="0.000104" iyy="8.3e-05" izz="7.6e-05" ixy="0.0" iyz="0.0" ixz="9e-06"/>
-    </inertial>
-    <visual>
-      <origin xyz="0.204017 0.24 -0.6215" rpy="0 0 0"/>
-      <geometry><mesh filename="file://$(find asump_description)/meshes/l1_us_mount.stl" scale="0.001 0.001 0.001"/></geometry>
-      <material name=""><color rgba="1 1 1 1"/></material>
-    </visual>
-    <collision>
-      <origin xyz="0.204017 0.24 -0.6215" rpy="0 0 0"/>
-      <geometry><mesh filename="file://$(find asump_description)/meshes/l1_us_mount.stl" scale="0.001 0.001 0.001"/></geometry>
-    </collision>
-  </link>
-  <joint name="l1_us_mount_joint" type="fixed">
-    <parent link="base_link"/>
-    <child link="l1_us_mount"/>
-    <origin xyz="0.0 0.0 0.0" rpy="0 0 0"/>
-  </joint>
-  <link name="l1_us_link">
-    <inertial>
-      <origin xyz="0.007108 0.000151 0.004104" rpy="0 0 0"/>
-      <mass value="0.052"/>
-      <inertia ixx="3e-06" iyy="3e-06" izz="3e-06" ixy="0.0" iyz="0.0" ixz="0.0"/>
-    </inertial>
-    <visual>
-      <origin xyz="0.238461 -0.234008 -0.318123" rpy="0 0 0"/>
-      <geometry><mesh filename="file://$(find asump_description)/meshes/l1_us_link.stl" scale="0.001 0.001 0.001"/></geometry>
-      <material name=""><color rgba="1 1 1 1"/></material>
-    </visual>
-    <collision>
-      <origin xyz="0.238461 -0.234008 -0.318123" rpy="0 0 0"/>
-      <geometry><mesh filename="file://$(find asump_description)/meshes/l1_us_link.stl" scale="0.001 0.001 0.001"/></geometry>
-    </collision>
-  </link>
-  <joint name="l1_us_sensor_joint" type="fixed">
-    <parent link="l1_us_mount"/>
-    <child link="l1_us_link"/>
-    <origin xyz="-0.034444 0.474008 -0.303377" rpy="0 0 0"/>
-  </joint>
-  <link name="fl_ultrasonic_link">
-    <inertial><origin xyz="3.8e-07 -0.007033 0.004235" rpy="0 0 0"/><mass value="0.052"/><inertia ixx="3e-06" iyy="3e-06" izz="3e-06" ixy="0.0" iyz="0.0" ixz="0.0"/></inertial>
-    <visual><origin xyz="0.091501 -0.460962 -0.319" rpy="0 0 0"/><geometry><mesh filename="file://$(find asump_description)/meshes/fl_ultrasonic_link.stl" scale="0.001 0.001 0.001"/></geometry><material name=""><color rgba="1 1 1 1"/></material></visual>
-    <collision><origin xyz="0.091501 -0.460962 -0.319" rpy="0 0 0"/><geometry><mesh filename="file://$(find asump_description)/meshes/fl_ultrasonic_link.stl" scale="0.001 0.001 0.001"/></geometry></collision>
-  </link>
-  <joint name="fl_ultrasonic_joint" type="fixed">
-    <parent link="face_sensors_mount_link"/>
-    <child link="fl_ultrasonic_link"/>
-    <origin xyz="-0.121493 0.028454 -0.0025" rpy="0 0 0"/>
-  </joint>
-  <link name="fr_ultrasonic_link">
-    <inertial><origin xyz="3.8e-07 -0.007033 0.004235" rpy="0 0 0"/><mass value="0.052"/><inertia ixx="3e-06" iyy="3e-06" izz="3e-06" ixy="0.0" iyz="0.0" ixz="0.0"/></inertial>
-    <visual><origin xyz="-0.151499 -0.460962 -0.319" rpy="0 0 0"/><geometry><mesh filename="file://$(find asump_description)/meshes/fr_ultrasonic_link.stl" scale="0.001 0.001 0.001"/></geometry><material name=""><color rgba="1 1 1 1"/></material></visual>
-    <collision><origin xyz="-0.151499 -0.460962 -0.319" rpy="0 0 0"/><geometry><mesh filename="file://$(find asump_description)/meshes/fr_ultrasonic_link.stl" scale="0.001 0.001 0.001"/></geometry></collision>
-  </link>
-  <joint name="fr_ultrasonic_joint" type="fixed">
-    <parent link="face_sensors_mount_link"/>
-    <child link="fr_ultrasonic_link"/>
-    <origin xyz="0.121507 0.028454 -0.0025" rpy="0 0 0"/>
-  </joint>
-  <link name="d435_link">
-    <inertial><origin xyz="0.244008 1.462543 -0.429365" rpy="0 0 0"/><mass value="0.343"/><inertia ixx="3.2e-05" iyy="0.000214" izz="0.000216" ixy="1e-06" iyz="0.0" ixz="0.0"/></inertial>
-    <visual><origin xyz="0.213596 1.008308 -0.751888" rpy="0 0 0"/><geometry><mesh filename="file://$(find asump_description)/meshes/d435_link.stl" scale="0.001 0.001 0.001"/></geometry><material name=""><color rgba="1 1 1 1"/></material></visual>
-    <collision><origin xyz="0.213596 1.008308 -0.751888" rpy="0 0 0"/><geometry><mesh filename="file://$(find asump_description)/meshes/d435_link.stl" scale="0.001 0.001 0.001"/></geometry></collision>
-  </link>
-  <joint name="d435_joint" type="fixed">
-    <parent link="face_sensors_mount_link"/>
-    <child link="d435_link"/>
-    <origin xyz="-0.243588 -1.440816 0.430388" rpy="0 0 0"/>
-  </joint> -->
+  <xacro:macro name="ultrasonic_mount" params="prefix xyz rpy">
+    <link name="${prefix}_us_mount_link">
+      <inertial>
+        <origin xyz="0 0 0" rpy="0 0 0"/>
+        <mass value="0.0437"/>
+        <inertia ixx="1.591e-5" ixy="0.0" ixz="-1.311e-6"
+                 iyy="1.267e-5" iyz="0.0"
+                 izz="1.167e-5"/>
+      </inertial>
+      <visual>
+        <origin xyz="0 0 0" rpy="0 0 0"/>
+        <geometry>
+          <mesh filename="file://$(find asump_description)/meshes/ultrasonic_mount.stl" scale="0.001 0.001 0.001"/>
+        </geometry>
+        <material name="plastic_material"><color rgba="0.85 0.85 0.85 1.0"/></material>
+      </visual>
+      <collision>
+        <origin xyz="0 0 0" rpy="0 0 0"/>
+        <geometry>
+          <mesh filename="file://$(find asump_description)/meshes/ultrasonic_mount.stl" scale="0.001 0.001 0.001"/>
+        </geometry>
+      </collision>
+    </link>
+    <joint name="${prefix}_us_mount_joint" type="fixed">
+      <parent link="body_link"/>
+      <child link="${prefix}_us_mount_link"/>
+      <origin xyz="${xyz}" rpy="${rpy}"/>
+    </joint>
+    <link name="${prefix}_us_sensor_link">
+      <inertial>
+        <origin xyz="0 0 0" rpy="0 0 0"/>
+        <mass value="0.0437"/>
+        <inertia ixx="1.591e-5" ixy="0.0" ixz="-1.311e-6"
+                 iyy="1.267e-5" iyz="0.0"
+                 izz="1.167e-5"/>
+      </inertial>
+      <visual>
+        <origin xyz="0 0 0" rpy="0 0 0"/>
+        <geometry>
+          <mesh filename="file://$(find asump_description)/meshes/ultrasonic_sensor.stl" scale="0.001 0.001 0.001"/>
+        </geometry>
+        <material name=""><color rgba="0.2 0.2 0.2 1.0"/></material>
+      </visual>
+      <collision>
+        <origin xyz="0 0 0" rpy="0 0 0"/>
+        <geometry>
+          <mesh filename="file://$(find asump_description)/meshes/ultrasonic_sensor.stl" scale="0.001 0.001 0.001"/>
+        </geometry>
+      </collision>
+    </link>
+    <joint name="${prefix}_us_sensor_joint" type="fixed">
+      <parent link="${prefix}_us_mount_link"/>
+      <child link="${prefix}_us_sensor_link"/>
+      <origin xyz="0.02845 0 0.018" rpy="0 0.5236 0"/>
+    </joint>
+  </xacro:macro>
+  <xacro:ultrasonic_mount prefix="left1" xyz="0.2615 0.24 0" rpy="0 0 1.5078" />
+  <xacro:ultrasonic_mount prefix="left2" xyz="-0.2995 0.24 0" rpy="0 0 1.5078" />
+  <xacro:ultrasonic_mount prefix="right1" xyz="0.2615 -0.24 0" rpy="0 0 -1.5078" />
+  <xacro:ultrasonic_mount prefix="right2" xyz="-0.2995 -0.24 0" rpy="0 0 -1.5078" />
+  <xacro:macro name="ultrasonic_mount_down" params="prefix xyz rpy">
+    <link name="${prefix}_us_mount_link">
+      <inertial>
+        <origin xyz="0 0 0" rpy="0 0 0"/>
+        <mass value="0.0437"/>
+        <inertia ixx="1.591e-5" ixy="0.0" ixz="-1.311e-6"
+                 iyy="1.267e-5" iyz="0.0"
+                 izz="1.167e-5"/>
+      </inertial>
+      <visual>
+        <origin xyz="0 0 0" rpy="0 0 0"/>
+        <geometry>
+          <mesh filename="file://$(find asump_description)/meshes/ultrasonic_mount_down.stl" scale="0.001 0.001 0.001"/>
+        </geometry>
+        <material name="plastic_material"><color rgba="0.85 0.85 0.85 1.0"/></material>
+      </visual>
+      <collision>
+        <origin xyz="0 0 0" rpy="0 0 0"/>
+        <geometry>
+          <mesh filename="file://$(find asump_description)/meshes/ultrasonic_mount_down.stl" scale="0.001 0.001 0.001"/>
+        </geometry>
+      </collision>
+    </link>
+    <joint name="${prefix}_us_mount_joint" type="fixed">
+      <parent link="body_link"/>
+      <child link="${prefix}_us_mount_link"/>
+      <origin xyz="${xyz}" rpy="${rpy}"/>
+    </joint>
+    <link name="${prefix}_us_sensor_link">
+      <inertial>
+        <origin xyz="0 0 0" rpy="0 0 0"/>
+        <mass value="0.0437"/>
+        <inertia ixx="1.591e-5" ixy="0.0" ixz="-1.311e-6"
+                 iyy="1.267e-5" iyz="0.0"
+                 izz="1.167e-5"/>
+      </inertial>
+      <visual>
+        <origin xyz="0 0 0" rpy="0 0 0"/>
+        <geometry>
+          <mesh filename="file://$(find asump_description)/meshes/ultrasonic_sensor.stl" scale="0.001 0.001 0.001"/>
+        </geometry>
+        <material name=""><color rgba="0.2 0.2 0.2 1.0"/></material>
+      </visual>
+      <collision>
+        <origin xyz="0 0 0" rpy="0 0 0"/>
+        <geometry>
+          <mesh filename="file://$(find asump_description)/meshes/ultrasonic_sensor.stl" scale="0.001 0.001 0.001"/>
+        </geometry>
+      </collision>
+    </link>
+    <joint name="${prefix}_us_sensor_joint" type="fixed">
+      <parent link="${prefix}_us_mount_link"/>
+      <child link="${prefix}_us_sensor_link"/>
+      <origin xyz="-0.022453 0 -0.028" rpy="0 2.0944 0"/>
+    </joint>
+  </xacro:macro>
+  <xacro:ultrasonic_mount_down prefix="back_left" xyz="-0.36 0.125 -0.03" rpy="0 0 0" />
+  <xacro:ultrasonic_mount_down prefix="back_right" xyz="-0.36 -0.125 -0.03" rpy="0 0 0" />
+  <link name="back_sensor_panel">
+    <inertial>
+      <origin xyz="0 0 0" rpy="0 0 0"/>
+      <mass value="0.4"/>
+      <inertia ixx="0.000511" iyy="0.011306" izz="0.011176" ixy="-3e-05" iyz="-2.8e-05" ixz="1.1e-05"/>
+    </inertial>
+    <visual>
+      <origin xyz="0 0 0" rpy="0 0 0"/>
+      <geometry><mesh filename="file://$(find asump_description)/meshes/back_sensor_panel.stl" scale="0.001 0.001 0.001"/></geometry>
+      <material name=""><color rgba="1 0.4318 0 1"/></material>
+    </visual>
+    <collision>
+      <origin xyz="0 0 0" rpy="0 0 0"/>
+      <geometry><mesh filename="file://$(find asump_description)/meshes/back_sensor_panel.stl" scale="0.001 0.001 0.001"/></geometry>
+    </collision>
+  </link>
+  <joint name="back_sensors_mount_joint" type="fixed">
+    <parent link="body_link"/>
+    <child link="back_sensor_panel"/>
+    <origin xyz="-0.3925 0.0 0.298" rpy="0 0 0"/>
+  </joint>
+  <xacro:sensor_d435 parent="back_sensor_panel" name="back_camera" use_nominal_extrinsics="true">
+    <origin xyz="-0.005 0 0.01" rpy="0 0 3.1415"/>
+  </xacro:sensor_d435>
+  <link name="cam_left_link">
+    <inertial>
+      <origin xyz="0 0 0" rpy="0 0 0"/>
+      <mass value="0.020"/>
+      <inertia ixx="1.0e-6" ixy="0.0" ixz="0.0"
+               iyy="5.4167e-7" iyz="0.0"
+               izz="5.4167e-7"/>
+    </inertial>
+    <visual>
+      <origin xyz="0 0 0" rpy="0 1.5707963 0"/>
+      <geometry>
+        <cylinder radius="0.010" length="0.005"/>
+      </geometry>
+      <material name="camera_material">
+        <color rgba="0.15 0.15 0.18 1.0"/>
+      </material>
+    </visual>
+    <collision>
+      <origin xyz="0 0 0" rpy="0 1.5707963 0"/>
+      <geometry>
+        <cylinder radius="0.010" length="0.005"/>
+      </geometry>
+    </collision>
+  </link>
+  <joint name="cam_left_joint" type="fixed">
+    <parent link="body_link"/>
+    <child link="cam_left_link"/>
+    <origin xyz="-0.2925 0.275 0.273" rpy="0 0 1.5708"/>
+  </joint>
+ <link name="cam_right_link">
+    <inertial>
+      <origin xyz="0 0 0" rpy="0 0 0"/>
+      <mass value="0.020"/>
+      <inertia ixx="1.0e-6" ixy="0.0" ixz="0.0"
+               iyy="5.4167e-7" iyz="0.0"
+               izz="5.4167e-7"/>
+    </inertial>
+    <visual>
+      <origin xyz="0 0 0" rpy="0 1.5707963 0"/>
+      <geometry>
+        <cylinder radius="0.010" length="0.005"/>
+      </geometry>
+      <material name="camera_material">
+        <color rgba="0.15 0.15 0.18 1.0"/>
+      </material>
+    </visual>
+    <collision>
+      <origin xyz="0 0 0" rpy="0 1.5707963 0"/>
+      <geometry>
+        <cylinder radius="0.010" length="0.005"/>
+      </geometry>
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